Commit message: S

File: ros_ws/src/lampo_description/urdf/sweepee/sweepee_diff.xacro (robot description, xacro)
@@ -24,10 +24,11 @@
           <origin xyz="0 0 0.2" rpy="0 0 0" />
           <mass value="250" />
-          <inertia ixx="12.0" ixy="0.0" ixz="0.0" iyy="12.0" iyz="0.0" izz="12.0" />
+          <!-- Solid-box approximation for 250 kg, 1.02 x 0.55 x 0.35 m -->
+          <inertia ixx="8.85" ixy="0.0" ixz="0.0" iyy="24.23" iyz="0.0" izz="27.98" />
       </inertial>
       <collision>
         <origin xyz="0 0 0.2" rpy="0 0 0" />
         <geometry>
-          <box size="0.3 ${base_y_size} 0.05"/>
+          <box size="${base_x_size} ${base_y_size} 0.05"/>
         </geometry>
       </collision>
@@ -52,16 +53,10 @@
       <origin xyz="${base_x_size/2-0.15} 0.0 ${base_z_size/2+0.085}" rpy="0 0 0" />
       <parent link="${prefix}base_link_sweepee" />
-      <child link="${prefix}front_laser" /> -->
-    </joint>
-      <link name="${prefix}rear_laser" />
-    <joint name="${prefix}rear_laser_joint" type="fixed">
-      <origin xyz="${-base_x_size/2+0.15} 0.0 ${base_z_size/2+0.085}" rpy="0 0 ${M_PI}" />
-      <parent link="${prefix}base_link_sweepee" />
-      <child link="${prefix}rear_laser" />
+      <child link="${prefix}front_laser" />
     </joint>
       <link name='${prefix}front_left_wheel'>
         <inertial>
           <mass value="5"/>
-          <inertia ixx="0.145"  ixy="0"  ixz="0" iyy="0.145" iyz="0" izz="0.125" />
+          <inertia ixx="0.014"  ixy="0"  ixz="0" iyy="0.014" iyz="0" izz="0.025" />
         </inertial>
         <visual>
@@ -79,5 +74,5 @@
         <inertial>
           <mass value="5"/>
-          <inertia ixx="0.145"  ixy="0"  ixz="0" iyy="0.145" iyz="0" izz="0.125" />
+          <inertia ixx="0.014"  ixy="0"  ixz="0" iyy="0.014" iyz="0" izz="0.025" />
         </inertial>
         <visual>
@@ -95,5 +90,5 @@
         <inertial>
           <mass value="5"/>
-          <inertia ixx="0.145"  ixy="0"  ixz="0" iyy="0.145" iyz="0" izz="0.125" />
+          <inertia ixx="0.014"  ixy="0"  ixz="0" iyy="0.014" iyz="0" izz="0.025" />
         </inertial>
         <visual>
@@ -111,5 +106,5 @@
         <inertial>
           <mass value="5"/>
-          <inertia ixx="0.145"  ixy="0"  ixz="0" iyy="0.145" iyz="0" izz="0.125" />
+          <inertia ixx="0.014"  ixy="0"  ixz="0" iyy="0.014" iyz="0" izz="0.025" />
         </inertial>
         <visual>
@@ -221,8 +216,8 @@
       </joint>
   <gazebo reference="${prefix}front_laser">
-    <sensor name='gpu_lidar' type='gpu_lidar'>"
+    <sensor name='gpu_lidar' type='gpu_lidar'>
         <pose relative_to='${prefix}front_laser'>0 0 0 0 0 0</pose>
         <gz_frame_id>${prefix}front_laser</gz_frame_id>
-        <topic>${prefix}lidar</topic>
+        <topic>${prefix}/lidar</topic>
         <update_rate>10</update_rate>
         <ray>
@@ -268,7 +263,7 @@
         <max_angular_velocity>1</max_angular_velocity>
         <min_angular_velocity>-1</min_angular_velocity>
-        <topic>${prefix}cmd_vel</topic>
+        <topic>${prefix}/cmd_vel</topic>
         <frame_id>${prefix}odom</frame_id>
-        <odom_topic>${prefix}odom</odom_topic>
+        <odom_topic>${prefix}/odom</odom_topic>
         <child_frame_id>${prefix}base_footprint</child_frame_id>
         <tf_topic>tf</tf_topic>

File: ros_ws/src/lampo_description/urdf/sweepee/sweepee_omni.xacro (robot description, xacro)
@@ -24,10 +24,11 @@
           <origin xyz="0 0 0.2" rpy="0 0 0" />
           <mass value="250" />
-          <inertia ixx="12.0" ixy="0.0" ixz="0.0" iyy="12.0" iyz="0.0" izz="12.0" />
+          <!-- Solid-box approximation for 250 kg, 1.02 x 0.55 x 0.35 m -->
+          <inertia ixx="8.85" ixy="0.0" ixz="0.0" iyy="24.23" iyz="0.0" izz="27.98" />
       </inertial>
       <collision>
         <origin xyz="0 0 0.2" rpy="0 0 0" />
         <geometry>
-          <box size="0.3 ${base_y_size} 0.05"/>
+          <box size="${base_x_size} ${base_y_size} 0.05"/>
         </geometry>
       </collision>
@@ -41,5 +42,5 @@
       <inertial>
         <mass value="5"/>
-        <inertia ixx="0.145"  ixy="0"  ixz="0" iyy="0.145" iyz="0" izz="0.125" />
+        <inertia ixx="0.014"  ixy="0"  ixz="0" iyy="0.014" iyz="0" izz="0.025" />
       </inertial>
       <visual>
@@ -52,5 +53,5 @@
       <origin xyz="${base_x_size/2-0.15} 0.0 ${base_z_size/2+0.085}" rpy="0 0 0" />
       <parent link="${prefix}base_link_sweepee" />
-      <child link="${prefix}front_laser" /> -->
+      <child link="${prefix}front_laser" />
     </joint>
     <gazebo reference='${prefix}front_laser_joint'>
@@ -61,5 +62,5 @@
       <inertial>
         <mass value="5"/>
-        <inertia ixx="0.145"  ixy="0"  ixz="0" iyy="0.145" iyz="0" izz="0.125" />
+        <inertia ixx="0.014"  ixy="0"  ixz="0" iyy="0.014" iyz="0" izz="0.025" />
       </inertial>
       <visual>
@@ -77,5 +78,5 @@
       <inertial>
         <mass value="5"/>
-        <inertia ixx="0.145"  ixy="0"  ixz="0" iyy="0.145" iyz="0" izz="0.125" />
+        <inertia ixx="0.014"  ixy="0"  ixz="0" iyy="0.014" iyz="0" izz="0.025" />
       </inertial>
       <visual>
@@ -93,5 +94,5 @@
       <inertial>
         <mass value="5"/>
-        <inertia ixx="0.145"  ixy="0"  ixz="0" iyy="0.145" iyz="0" izz="0.125" />
+        <inertia ixx="0.014"  ixy="0"  ixz="0" iyy="0.014" iyz="0" izz="0.025" />
       </inertial>
       <visual>
@@ -109,5 +110,5 @@
       <inertial>
         <mass value="5"/>
-        <inertia ixx="0.145"  ixy="0"  ixz="0" iyy="0.145" iyz="0" izz="0.125" />
+        <inertia ixx="0.014"  ixy="0"  ixz="0" iyy="0.014" iyz="0" izz="0.025" />
       </inertial>
       <visual>
@@ -213,5 +214,5 @@
       <sensor name='gpu_lidar' type='gpu_lidar'>
           <pose relative_to='${prefix}front_laser'>0 0 0 0 0 0</pose>
-          <frame_id>${prefix}front_laser</frame_id>
+          <gz_frame_id>${prefix}front_laser</gz_frame_id>
           <topic>${prefix}/lidar</topic>
           <update_rate>10</update_rate>
