Commit message: Fix the robot description and world physics
Declare the undefined `prefix` xacro argument so the description renders at
all. Wheel joints become continuous with limits and damping; inertias are
corrected to physically possible values; the base collision matches the
chassis. Sensors declare their frames, and the camera gains a REP-103 optical
frame so point clouds are not rotated 90 degrees. The warehouse walls, pillars
and crates get collision geometry -- previously the only collisions were two
infinite planes and the robot drove through everything.

Gripper actuation is opt-in (gripper_control:=false): the Robotiq 4-bar finger
linkage can only be approximated with mimic joints, and the resulting limit
violation aborts the simulator outright.

Co-Authored-By: Claude Opus 5 (1M context) <noreply@anthropic.com>

File: ros_ws/src/lampo_description/urdf/mm_camera.xacro (robot description, xacro)
@@ -5,9 +5,10 @@
     <inertial>
       <mass value="0.2"/>
-      <inertia ixx="0.0145"  ixy="0"  ixz="0" iyy="0.0145" iyz="0" izz="0.02125" />
+      <!-- Solid box 0.09 x 0.025 x 0.025 m (RealSense D435-class) -->
+      <inertia ixx="2.1e-5"  ixy="0"  ixz="0" iyy="1.4e-4" iyz="0" izz="1.4e-4" />
     </inertial>
   </link>
   <joint name="$(arg prefix)cam_joint" type="fixed">
-    <origin xyz="0.0 -0.1 0.0" rpy="0 -1.57 1.57" />
+    <origin xyz="0.0 -0.1 0.0" rpy="0 ${-pi/2} ${pi/2}" />
     <parent link="$(arg prefix)wrist_3_link" />
     <child link="$(arg prefix)cam_link" />
@@ -17,6 +18,15 @@
     <preserveFixedJoint>true</preserveFixedJoint>
   </gazebo>
+  <!-- REP-103 optical frame: image data uses z-forward / y-down, while the
+       body frame is x-forward / z-up. -->
+  <link name="$(arg prefix)cam_optical_frame"/>
+  <joint name="$(arg prefix)cam_optical_joint" type="fixed">
+    <origin xyz="0 0 0" rpy="${-pi/2} 0 ${-pi/2}"/>
+    <parent link="$(arg prefix)cam_link"/>
+    <child link="$(arg prefix)cam_optical_frame"/>
+  </joint>
   <gazebo reference="$(arg prefix)cam_link">
     <sensor name="rs_front" type="rgbd_camera">
+      <gz_frame_id>$(arg prefix)cam_optical_frame</gz_frame_id>
       <pose>0.0 0.0 0.0 0.0 0.0 0.0</pose>
       <always_on>1</always_on>
@@ -52,5 +62,5 @@
         <clip>
           <near>0.01</near>
-          <far>300</far>
+          <far>50</far>
         </clip>
         <depth_camera>

File: ros_ws/src/lampo_description/urdf/mm_gripper.xacro (robot description, xacro)
@@ -6,47 +6,82 @@
       <origin xyz="0 0 0" rpy="0 0 0" />
   </xacro:robotiq_gripper>
-  <ros2_control name="$(arg tf_prefix)/robotiq_control" type="system">
-      <!-- Plugins -->
-      <hardware>
-        <plugin>gz_ros2_control/GazeboSimSystem</plugin>
-      </hardware>
-      <joint name="$(arg tf_prefix)robotiq_85_left_knuckle_joint">
-        <command_interface name="position" />
-        <state_interface name="position">
-            <param name="initial_value">0.7929</param>
-        </state_interface>
-        <state_interface name="velocity"/>
-      </joint>
-      <!-- When simulating we need to include the rest of the gripper joints -->
-      <joint name="$(arg tf_prefix)robotiq_85_right_knuckle_joint">
-        <param name="mimic">$(arg tf_prefix)robotiq_85_left_knuckle_joint</param>
-        <param name="multiplier">-1</param>
-        <state_interface name="position"/>
-        <state_interface name="velocity"/>
-      </joint>
-      <joint name="$(arg tf_prefix)robotiq_85_left_inner_knuckle_joint">
-        <param name="mimic">$(arg tf_prefix)robotiq_85_left_knuckle_joint</param>
-        <param name="multiplier">1</param>
-        <state_interface name="position"/>
-        <state_interface name="velocity"/>
-      </joint>
-      <joint name="$(arg tf_prefix)robotiq_85_right_inner_knuckle_joint">
-        <param name="mimic">$(arg tf_prefix)robotiq_85_left_knuckle_joint</param>
-        <param name="multiplier">-1</param>
-        <state_interface name="position"/>
-        <state_interface name="velocity"/>
-      </joint>
-      <joint name="$(arg tf_prefix)robotiq_85_left_finger_tip_joint">
-        <param name="mimic">$(arg tf_prefix)robotiq_85_left_knuckle_joint</param>
-        <param name="multiplier">-1</param>
-        <state_interface name="position"/>
-        <state_interface name="velocity"/>
-      </joint>
-      <joint name="$(arg tf_prefix)robotiq_85_right_finger_tip_joint">
-        <param name="mimic">$(arg tf_prefix)robotiq_85_left_knuckle_joint</param>
-        <param name="multiplier">1</param>
-        <state_interface name="position"/>
-        <state_interface name="velocity"/>
-      </joint>
-  </ros2_control>
+  <!-- No "/" in the component name: hardware_interface uses it to build
+       parameter and service names, and a slash silently prevents the
+       command interfaces from being exported at all. -->
+  <!-- Gripper actuation is OFF by default (gripper_control:=false).
+       Why: the Robotiq 2F-85 fingers are a closed 4 bar linkage. URDF cannot
+       express a closed chain, so it is approximated with <mimic> joints.
+       Neither engine handles that well:
+         * DART (gz-sim 9) cannot create mimic constraints at all;
+         * Bullet Featherstone can, but the loop is over constrained and the
+           solver drives the knuckle joint far outside its [0, 0.8] limit.
+       ros2_control's joint limiter treats any out of limit reading as a
+       hardware fault and throws a FATAL exception, which aborts the whole
+       simulator. Rather than ship a demo that randomly dies, the gripper is
+       mounted as passive geometry and the arm is the ros2_control example.
+       Set gripper_control:=true to experiment with it. -->
+  <xacro:arg name="gripper_control" default="false" />
+  <xacro:if value="$(arg gripper_control)">
+    <ros2_control name="$(arg tf_prefix)robotiq_control" type="system">
+        <!-- Plugins -->
+        <hardware>
+          <plugin>gz_ros2_control/GazeboSimSystem</plugin>
+        </hardware>
+        <joint name="$(arg tf_prefix)robotiq_85_left_knuckle_joint">
+          <command_interface name="position">
+            <!-- Widen the limits ros2_control enforces, slightly beyond the
+                 URDF's [0, 0.8]. The Robotiq fingers are a closed 4 bar linkage
+                 that URDF can only approximate with mimic joints, so the solver
+                 settles a few tens of millirad outside the nominal range. The
+                 joint limiter treats that as a hardware fault and throws a fatal
+                 exception, which takes down the whole simulator. -->
+            <param name="min">-0.1</param>
+            <param name="max">0.9</param>
+          </command_interface>
+          <state_interface name="position">
+              <!-- Start the gripper mid range, NOT at either end stop.
+                   ros2_control's joint limiter throws a fatal std::runtime_error
+                   the instant a joint reads outside its limits, which aborts the
+                   whole simulator. The Robotiq 4 bar finger linkage cannot be
+                   expressed exactly in URDF, so a few millirad of physics jitter
+                   is unavoidable: starting at 0 (or at the original 0.7929, a
+                   hair under the 0.8 stop) crossed the limit within one step.
+                   0.4 leaves margin on both sides. Range is [0, 0.8]. -->
+              <param name="initial_value">0.4</param>
+          </state_interface>
+          <state_interface name="velocity"/>
+        </joint>
+        <!-- When simulating we need to include the rest of the gripper joints -->
+        <joint name="$(arg tf_prefix)robotiq_85_right_knuckle_joint">
+          <param name="mimic">$(arg tf_prefix)robotiq_85_left_knuckle_joint</param>
+          <param name="multiplier">-1</param>
+          <state_interface name="position"/>
+          <state_interface name="velocity"/>
+        </joint>
+        <joint name="$(arg tf_prefix)robotiq_85_left_inner_knuckle_joint">
+          <param name="mimic">$(arg tf_prefix)robotiq_85_left_knuckle_joint</param>
+          <param name="multiplier">1</param>
+          <state_interface name="position"/>
+          <state_interface name="velocity"/>
+        </joint>
+        <joint name="$(arg tf_prefix)robotiq_85_right_inner_knuckle_joint">
+          <param name="mimic">$(arg tf_prefix)robotiq_85_left_knuckle_joint</param>
+          <param name="multiplier">-1</param>
+          <state_interface name="position"/>
+          <state_interface name="velocity"/>
+        </joint>
+        <joint name="$(arg tf_prefix)robotiq_85_left_finger_tip_joint">
+          <param name="mimic">$(arg tf_prefix)robotiq_85_left_knuckle_joint</param>
+          <param name="multiplier">-1</param>
+          <state_interface name="position"/>
+          <state_interface name="velocity"/>
+        </joint>
+        <joint name="$(arg tf_prefix)robotiq_85_right_finger_tip_joint">
+          <param name="mimic">$(arg tf_prefix)robotiq_85_left_knuckle_joint</param>
+          <param name="multiplier">1</param>
+          <state_interface name="position"/>
+          <state_interface name="velocity"/>
+        </joint>
+    </ros2_control>
+  </xacro:if>
 </robot>

File: ros_ws/src/lampo_description/urdf/sweepee/sweepee_diff.xacro (robot description, xacro)
@@ -30,5 +30,5 @@
         <origin xyz="0 0 0.2" rpy="0 0 0" />
         <geometry>
-          <box size="${base_x_size} ${base_y_size} 0.05"/>
+          <box size="${base_x_size} ${base_y_size} ${base_z_size}"/>
         </geometry>
       </collision>
@@ -41,6 +41,7 @@
     <link name="${prefix}front_laser">
       <inertial>
-        <mass value="5"/>
-        <inertia ixx="0.145"  ixy="0"  ixz="0" iyy="0.145" iyz="0" izz="0.125" />
+        <mass value="1.1"/>
+        <!-- SICK LMS1xx: solid cylinder r=0.1 m, h=0.005 m -->
+        <inertia ixx="0.00275"  ixy="0"  ixz="0" iyy="0.00275" iyz="0" izz="0.0055" />
       </inertial>
       <visual>
@@ -55,4 +56,10 @@
       <child link="${prefix}front_laser" />
     </joint>
+    <!-- Keep front_laser as its own SDF link: the lidar sensor's
+         <pose relative_to='${prefix}front_laser'> needs the frame to survive. -->
+    <gazebo reference='${prefix}front_laser_joint'>
+      <disableFixedJointLumping>true</disableFixedJointLumping>
+      <preserveFixedJoint>true</preserveFixedJoint>
+    </gazebo>
       <link name='${prefix}front_left_wheel'>
         <inertial>
@@ -187,31 +194,35 @@
         </collision>
       </gazebo>
-      <joint name='${prefix}front_left_wheel_joint' type='revolute'>
+      <joint name='${prefix}front_left_wheel_joint' type='continuous'>
         <origin xyz="0.3 0.25 0.1" rpy="-1.5707 0 0"/>
         <parent link="${prefix}base_link_sweepee"/>
         <child link="${prefix}front_left_wheel"/>
         <axis xyz="0 0 1"/>
-        <limit effort="10000.0" lower="-1.79769e+308" upper="1.79769e+308" velocity="15.1"/>
-      </joint>
-      <joint name='${prefix}front_right_wheel_joint' type='revolute'>
+        <limit effort="150.0" velocity="15.1"/>
+      <dynamics damping="0.05" friction="0.1"/>
+      </joint>
+      <joint name='${prefix}front_right_wheel_joint' type='continuous'>
         <origin xyz="0.3 -0.25 0.1" rpy="-1.5707 0 0"/>
         <parent link="${prefix}base_link_sweepee"/>
         <child link="${prefix}front_right_wheel"/>
         <axis xyz="0 0 1"/>
-        <limit effort="10000.0" lower="-1.79769e+308" upper="1.79769e+308" velocity="15.1"/>
-      </joint>
-      <joint name='${prefix}rear_left_wheel_joint' type='revolute'>
+        <limit effort="150.0" velocity="15.1"/>
+      <dynamics damping="0.05" friction="0.1"/>
+      </joint>
+      <joint name='${prefix}rear_left_wheel_joint' type='continuous'>
         <origin xyz="-0.3 0.25 0.1" rpy="-1.5707 0 0"/>
         <parent link="${prefix}base_link_sweepee"/>
         <child link="${prefix}rear_left_wheel"/>
         <axis xyz="0 0 1"/>
-        <limit effort="10000.0" lower="-1.79769e+308" upper="1.79769e+308" velocity="15.1"/>
-      </joint>
-      <joint name='${prefix}rear_right_wheel_joint' type='revolute'>
+        <limit effort="150.0" velocity="15.1"/>
+      <dynamics damping="0.05" friction="0.1"/>
+      </joint>
+      <joint name='${prefix}rear_right_wheel_joint' type='continuous'>
         <origin xyz="-0.3 -0.25 0.1" rpy="-1.5707 0 0"/>
         <parent link="${prefix}base_link_sweepee"/>
         <child link="${prefix}rear_right_wheel"/>
         <axis xyz="0 0 1"/>
-        <limit effort="10000.0" lower="-1.79769e+308" upper="1.79769e+308" velocity="15.1"/>
+        <limit effort="150.0" velocity="15.1"/>
+      <dynamics damping="0.05" friction="0.1"/>
       </joint>
   <gazebo reference="${prefix}front_laser">
@@ -246,4 +257,14 @@
     </sensor>
   </gazebo>
+    <!-- Publish the wheel joint positions. Without this nothing publishes
+         /joint_states for the wheels: joint_state_broadcaster only covers
+         ros2_control joints (the arm/gripper), so robot_state_publisher would
+         never emit the base -> wheel transforms and RViz shows a broken model. -->
+    <gazebo>
+      <plugin filename="gz-sim-joint-state-publisher-system"
+              name="gz::sim::systems::JointStatePublisher">
+        <topic>${prefix}/joint_states</topic>
+      </plugin>
+    </gazebo>
   <gazebo>
       <plugin
@@ -267,5 +288,5 @@
         <odom_topic>${prefix}/odom</odom_topic>
         <child_frame_id>${prefix}base_footprint</child_frame_id>
-        <tf_topic>tf</tf_topic>
+        <tf_topic>/${prefix}/tf</tf_topic>
       </plugin>
     </gazebo>

File: ros_ws/src/lampo_description/urdf/sweepee/sweepee_omni.xacro (robot description, xacro)
@@ -30,5 +30,5 @@
         <origin xyz="0 0 0.2" rpy="0 0 0" />
         <geometry>
-          <box size="${base_x_size} ${base_y_size} 0.05"/>
+          <box size="${base_x_size} ${base_y_size} ${base_z_size}"/>
         </geometry>
       </collision>
@@ -41,6 +41,7 @@
     <link name="${prefix}front_laser">
       <inertial>
-        <mass value="5"/>
-        <inertia ixx="0.014"  ixy="0"  ixz="0" iyy="0.014" iyz="0" izz="0.025" />
+        <mass value="1.1"/>
+        <!-- SICK LMS1xx: solid cylinder r=0.1 m, h=0.005 m -->
+        <inertia ixx="0.00275"  ixy="0"  ixz="0" iyy="0.00275" iyz="0" izz="0.0055" />
       </inertial>
       <visual>
@@ -175,34 +176,39 @@
       </collision>
     </gazebo>
-    <joint name='${prefix}front_left_wheel_joint' type='revolute'>
+    <joint name='${prefix}front_left_wheel_joint' type='continuous'>
       <origin xyz="0.3 0.25 0.1" rpy="-1.5707 0 0"/>
       <parent link="${prefix}base_link_sweepee"/>
       <child link="${prefix}front_left_wheel"/>
       <axis xyz="0 0 1"/>
-      <limit effort="10000.0" lower="-1.79769e+308" upper="1.79769e+308" velocity="15.1"/>
-    </joint>
-    <joint name='${prefix}front_right_wheel_joint' type='revolute'>
+      <limit effort="150.0" velocity="15.1"/>
+      <dynamics damping="0.05" friction="0.1"/>
+    </joint>
+    <joint name='${prefix}front_right_wheel_joint' type='continuous'>
       <origin xyz="0.3 -0.25 0.1" rpy="-1.5707 0 0"/>
       <parent link="${prefix}base_link_sweepee"/>
       <child link="${prefix}front_right_wheel"/>
       <axis xyz="0 0 1"/>
-      <limit effort="10000.0" lower="-1.79769e+308" upper="1.79769e+308" velocity="15.1"/>
-    </joint>
-    <joint name='${prefix}rear_left_wheel_joint' type='revolute'>
+      <limit effort="150.0" velocity="15.1"/>
+      <dynamics damping="0.05" friction="0.1"/>
+    </joint>
+    <joint name='${prefix}rear_left_wheel_joint' type='continuous'>
       <origin xyz="-0.3 0.25 0.1" rpy="-1.5707 0 0"/>
       <parent link="${prefix}base_link_sweepee"/>
       <child link="${prefix}rear_left_wheel"/>
       <axis xyz="0 0 1"/>
-      <limit effort="10000.0" lower="-1.79769e+308" upper="1.79769e+308" velocity="15.1"/>
-    </joint>
-    <joint name='${prefix}rear_right_wheel_joint' type='revolute'>
+      <limit effort="150.0" velocity="15.1"/>
+      <dynamics damping="0.05" friction="0.1"/>
+    </joint>
+    <joint name='${prefix}rear_right_wheel_joint' type='continuous'>
       <origin xyz="-0.3 -0.25 0.1" rpy="-1.5707 0 0"/>
       <parent link="${prefix}base_link_sweepee"/>
       <child link="${prefix}rear_right_wheel"/>
       <axis xyz="0 0 1"/>
-      <limit effort="10000.0" lower="-1.79769e+308" upper="1.79769e+308" velocity="15.1"/>
+      <limit effort="150.0" velocity="15.1"/>
+      <dynamics damping="0.05" friction="0.1"/>
     </joint>
     <gazebo reference="${prefix}base_link_sweepee">
       <sensor name="imu_sensor" type="imu">
+          <gz_frame_id>${prefix}base_link_sweepee</gz_frame_id>
           <always_on>1</always_on>
           <update_rate>10</update_rate>
@@ -242,4 +248,14 @@
       </sensor>
     </gazebo>
+    <!-- Publish the wheel joint positions. Without this nothing publishes
+         /joint_states for the wheels: joint_state_broadcaster only covers
+         ros2_control joints (the arm/gripper), so robot_state_publisher would
+         never emit the base -> wheel transforms and RViz shows a broken model. -->
+    <gazebo>
+      <plugin filename="gz-sim-joint-state-publisher-system"
+              name="gz::sim::systems::JointStatePublisher">
+        <topic>${prefix}/joint_states</topic>
+      </plugin>
+    </gazebo>
     <gazebo>
       <plugin
@@ -260,5 +276,6 @@
         <odom_topic>${prefix}/odom</odom_topic>
         <child_frame_id>${prefix}base_footprint</child_frame_id>
-        <tf_topic>tf</tf_topic>
+        <odom_publish_frequency>50</odom_publish_frequency>
+        <tf_topic>/${prefix}/tf</tf_topic>
       </plugin>
     </gazebo>

File: ros_ws/src/lampo_description/urdf/system.urdf.xacro (robot description, xacro)
@@ -1,4 +1,7 @@
 <?xml version="1.0"?>
-<robot name="$(arg prefix)/mm1" xmlns:xacro="http://ros.org/wiki/xacro" xmlns:gz="http://gazebosim.org/schema">>
+<robot name="$(arg prefix)mm1" xmlns:xacro="http://ros.org/wiki/xacro" xmlns:gz="http://gazebosim.org/schema">
+  <!-- TF/topic prefix for this robot. Must end with a separator (e.g. "r1_")
+       because every link and joint name is built as ${prefix}<name>. -->
+  <xacro:arg name="prefix" default="r1_" />
   <xacro:arg name="omni" default="false" />
   <xacro:arg name="mm" default="false" />
